File: project_kicad/project_design.kicad_pcb (KiCad board)
At the start: 2 copper layers, 27 parts, among them J1 Screw_Terminal_01x02, J2 USB_C_Receptacle_PowerOnly_6P, U2 NSL-32, U3 CJ432

Commit message: cad
Parts:
- added Cin1: 22uF, footprints:400PK22MEFC12.5X20, F.Cu at (221.0, 106.7)
- added Cin2: 22uF, footprints:400PK22MEFC12.5X20, F.Cu at (205.8, 106.7)
- added Rcs1: 910m, footprints:CRCW04021K07FKED, F.Cu at (201.2, 116.2)
Connections:
- D2 pad 2: Net-(C2-Pad1) -> Net-(D2-Pad2)
- L1 pad 1: Net-(C1-Pad1) -> Net-(D1-Pad1)
- L1 pad 2: Net-(C2-Pad1) -> Net-(D2-Pad2)
