File: project_kicad/project_design.kicad_sch (KiCad schematic)
At the start: 31 parts, among them J1 Screw_Terminal_01x02, J2 USB_C_Receptacle_PowerOnly_6P, Q1 Q_NMOS_DGS, T1 Transformer_1P_2S, U1 UCC28740, U2 NSL-32, U3 CJ432

Commit message: cad
Parts:
- removed C1: 22uF, symbol Device:C
- removed C2: 22uF, Capacitor_SMD:C_0603_1608Metric_Pad1.08x0.95mm_HandSolder, symbol Device:C
- removed R2: 910m, Resistor_SMD:R_0201_0603Metric_Pad0.64x0.40mm_HandSolder, symbol Device:R
- added Cin1, Cin2: 22uF, footprints:400PK22MEFC12.5X20, symbol 400PK22MEFC12.5X20:400PK22MEFC12.5X20
- added Rcs1: 910m, footprints:CRCW04021K07FKED, symbol CRCW040234K0FKED:CRCW040234K0FKEDHP
- D2: footprint (none) -> Diode_SMD:D_0201_0603Metric_Pad0.64x0.40mm_HandSolder
- D3: footprint (none) -> Diode_SMD:D_0402_1005Metric_Pad0.77x0.64mm_HandSolder
- J1: footprint (none) -> TerminalBlock_MetzConnect:TerminalBlock_MetzConnect_Type703_RT10N02HGLU_1x02_P9.52mm_Horizontal
- J2: footprint (none) -> Connector_USB:USB_C_Plug_Molex_105444
- L1: footprint (none) -> Inductor_SMD:L_0201_0603Metric_Pad0.64x0.40mm_HandSolder
- R1: footprint (none) -> Resistor_SMD:R_0201_0603Metric_Pad0.64x0.40mm_HandSolder
Connections:
- net Earth: now also Cin1.2, Cin2.2, Rcs1.1
- net at D2.2 (A), L1.2, T1.6 (SD)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: now also Cin2.1
- net at Q1.3 (S), R3.1: now also Rcs1.2
- net at D1.1 (+), L1.1: now also Cin1.1

Commit message: merge
Parts:
- removed J1: Screw_Terminal_01x02, TerminalBlock_MetzConnect:TerminalBlock_MetzConnect_Type703_RT10N02HGLU_1x02_P9.52mm_Horizontal, symbol Connector:Screw_Terminal_01x02
- removed J2: USB_C_Receptacle_PowerOnly_6P, Connector_USB:USB_C_Plug_Molex_105444, symbol Connector:USB_C_Receptacle_PowerOnly_6P
- added V1: VSIN, symbol Simulation_SPICE:VSIN
- R1: value R -> 10; Spice_Model (none) -> 10; Spice_Netlist_Enabled (none) -> Y; Spice_Primitive (none) -> R
Connections:
- net Earth: no longer C6.1, R12.1, T1.1 (AA), U3.3 (A)
- net at R1.1: now also V1.1
- net at D1.4: now also V1.2
- new net GND: C6.1, R12.1, T1.1 (AA), U3.3 (A)
- no-connect marks 3 -> 0
